File: Electrical/Connectors.sch (KiCad schematic (older format))
At the start: 7 parts

Commit message: Continued work on schematic
Parts:
- gave numbers to parts that had none: 7
Other:
- note removed: "reverse input protection"
- moved on the sheet: C22, C23, CON1, P1, P2, P3, P4

Commit message: schematic 95% done
Parts:
- removed C22, C23: C, symbol C
- added C22, C23: 100uF, Capacitors_SMD:c_elec_5x5.3, symbol CP1
- added U7: SN74AHCT125, Housings_SSOP:TSSOP-14_4.4x5mm_Pitch0.65mm, symbol SN74AHCT125
- CON1: footprint (none) -> Connect:BARREL_JACK
- P1: footprint (none) -> Connectors_JST:JST_PH_B2B-PH-K_02x2.00mm_Straight
- P2: footprint (none) -> Connectors_JST:JST_PH_B5B-PH-K_05x2.00mm_Straight
- P3, P4: footprint (none) -> Connectors_JST:JST_PH_B3B-PH-K_03x2.00mm_Straight
Connections:
- net +5V: now also C22.1, C23.1, U7.14 (VCC)
- net GND: now also CON1.2, CON1.3, C22.2, C23.2, U7.1 (1OE), U7.4 (2OE), U7.7 (GND)
- net LED_CTRL: now also U7.2 (1A), U7.5 (2A)
- net LED_out1: now reaches P3.2 (P2)
- net LED_out1: now also U7.3 (1Y)
- net LED_out2: now reaches P4.2 (P2)
- net LED_out2: now also U7.6 (2Y)
- net +12V: now reaches CON1.1
Other:
- moved on the sheet: P3, P4

Commit message: minor tweaks
Parts:
- added C30: 1uF, Capacitors_SMD:C_0603, symbol C
Connections:
- net +5V: now also C30.1
- net GND: now also C30.2
- no-connect marks 0 -> 6
Changed lines of the file:
@@
 3.3V_IN
 $Comp
-L +5V #PWR033
+L +5V #PWR034
 U 1 1 584A1D9A
 P 9550 2250
-F 0 "#PWR033" H 9550 2100 50  0001 C CNN
+F 0 "#PWR034" H 9550 2100 50  0001 C CNN
 F 1 "+5V" H 9550 2390 50  0000 C CNN
 F 2 "" H 9550 2250 50  0000 C CNN
@@
 $EndComp
 $Comp
-L +3.3V #PWR034
+L +3.3V #PWR035
 U 1 1 584A1DB8
 P 5150 4300
-F 0 "#PWR034" H 5150 4150 50  0001 C CNN
+F 0 "#PWR035" H 5150 4150 50  0001 C CNN
 F 1 "+3.3V" H 5150 4440 50  0000 C CNN
 F 2 "" H 5150 4300 50  0000 C CNN
@@
 $EndComp
 $Comp
-L GND #PWR035
+L GND #PWR036
 U 1 1 584A1DD6
 P 5150 4900
-F 0 "#PWR035" H 5150 4650 50  0001 C CNN
+F 0 "#PWR036" H 5150 4650 50  0001 C CNN
 F 1 "GND" H 5150 4750 50  0000 C CNN
 F 2 "" H 5150 4900 50  0000 C CNN
@@
 $EndComp
 $Comp
-L +BATT #PWR036
+L +BATT #PWR037
 U 1 1 584A1F38
 P 4850 3000
-F 0 "#PWR036" H 4850 2850 50  0001 C CNN
+F 0 "#PWR037" H 4850 2850 50  0001 C CNN
 F 1 "+BATT" H 4850 3140 50  0000 C CNN
 F 2 "" H 4850 3000 50  0000 C CNN
@@
 $EndComp
 $Comp
-L GND #PWR037
+L GND #PWR038
 U 1 1 584A20CB
 P 4850 3300
-F 0 "#PWR037" H 4850 3050 50  0001 C CNN
+F 0 "#PWR038" H 4850 3050 50  0001 C CNN
 F 1 "GND" H 4850 3150 50  0000 C CNN
 F 2 "" H 4850 3300 50  0000 C CNN
@@
 $EndComp
 $Comp
-L GND #PWR038
+L GND #PWR039
 U 1 1 584A23C4
 P 9550 2650
-F 0 "#PWR038" H 9550 2400 50  0001 C CNN
+F 0 "#PWR039" H 9550 2400 50  0001 C CNN
 F 1 "GND" H 9550 2500 50  0000 C CNN
 F 2 "" H 9550 2650 50  0000 C CNN
@@
 $EndComp
 $Comp
-L GND #PWR039
+L GND #PWR040
 U 1 1 584A2415
 P 9550 3550
-F 0 "#PWR039" H 9550 3300 50  0001 C CNN
+F 0 "#PWR040" H 9550 3300 50  0001 C CNN
 F 1 "GND" H 9550 3400 50  0000 C CNN
 F 2 "" H 9550 3550 50  0000 C CNN
@@
 $EndComp
 $Comp
-L +5V #PWR040
+L +5V #PWR041
 U 1 1 584A2510
 P 9550 3150
-F 0 "#PWR040" H 9550 3000 50  0001 C CNN
+F 0 "#PWR041" H 9550 3000 50  0001 C CNN
 F 1 "+5V" H 9550 3290 50  0000 C CNN
 F 2 "" H 9550 3150 50  0000 C CNN
@@
 $EndComp
 $Comp
-L +BATT #PWR041
+L +BATT #PWR042
 U 1 1 584A2723
 P 1100 800
-F 0 "#PWR041" H 1100 650 50  0001 C CNN
+F 0 "#PWR042" H 1100 650 50  0001 C CNN
 F 1 "+BATT" H 1100 940 50  0000 C CNN
 F 2 "" H 1100 800 50  0000 C CNN
@@
 $EndComp
 $Comp
-L +3.3V #PWR042
+L +3.3V #PWR043
 U 1 1 584A2854
 P 1750 800
-F 0 "#PWR042" H 1750 650 50  0001 C CNN
+F 0 "#PWR043" H 1750 650 50  0001 C CNN
 F 1 "+3.3V" H 1750 940 50  0000 C CNN
 F 2 "" H 1750 800 50  0000 C CNN
@@
 Battery Input Connection
 $Comp
-L +5V #PWR043
+L +5V #PWR044
 U 1 1 584A339B
 P 1750 1200
-F 0 "#PWR043" H 1750 1050 50  0001 C CNN
+F 0 "#PWR044" H 1750 1050 50  0001 C CNN
 F 1 "+5V" H 1750 1340 50  0000 C CNN
 F 2 "" H 1750 1200 50  0000 C CNN
@@
 input protection?
 $Comp
-L GND #PWR044
+L GND #PWR045
 U 1 1 5859BE29
 P 7250 4800
-F 0 "#PWR044" H 7250 4550 50  0001 C CNN
+F 0 "#PWR045" H 7250 4550 50  0001 C CNN
 F 1 "GND" H 7250 4650 50  0000 C CNN
 F 2 "" H 7250 4800 50  0000 C CNN
@@
 $EndComp
 $Comp
-L +12V #PWR045
+L +12V #PWR046
 U 1 1 5859BEAB
 P 7250 4400
-F 0 "#PWR045" H 7250 4250 50  0001 C CNN
+F 0 "#PWR046" H 7250 4250 50  0001 C CNN
 F 1 "+12V" H 7250 4540 50  0000 C CNN
 F 2 "" H 7250 4400 50  0000 C CNN
 F 3 "" H 7250 4400 50  0000 C CNN
 	1    7250 4400
-	1    0    0    -1
-$EndComp
-$Comp
-L +12V #PWR046
-U 1 1 5859BF08
-P 1100 1200
-F 0 "#PWR046" H 1100 1050 50  0001 C CNN
-F 1 "+12V" H 1100 1340 50  0000 C CNN
-F 2 "" H 1100 1200 50  0000 C CNN
-F 3 "" H 1100 1200 50  0000 C CNN
-	1    1100 1200
 	1    0    0    -1
 $EndComp
@@
 L +5V #PWR047
 U 1 1 5859F883
-P 8450 2500
-F 0 "#PWR047" H 8450 2350 50  0001 C CNN
-F 1 "+5V" H 8450 2640 50  0000 C CNN
-F 2 "" H 8450 2500 50  0000 C CNN
-F 3 "" H 8450 2500 50  0000 C CNN
-	1    8450 2500
+P 8500 2500
+F 0 "#PWR047" H 8500 2350 50  0001 C CNN
+F 1 "+5V" H 8500 2640 50  0000 C CNN
+F 2 "" H 8500 2500 50  0000 C CNN
+F 3 "" H 8500 2500 50  0000 C CNN
+	1    8500 2500
 	1    0    0    -1
 $EndComp
@@
 	7250 4500 7100 4500
 Wire Wire Line
-	1100 1200 1100 1300
-Wire Wire Line
-	1100 1300 900  1300
-Wire Wire Line
-	8450 2500 8450 2600
-Wire Wire Line
-	8450 2600 8350 2600
+	8500 2500 8500 2650
+Wire Wire Line
+	8350 2600 8500 2600
 Wire Wire Line
 	6750 3200 6850 3200
@@
 Wire Wire Line
 	8800 2250 8800 2300
+Wire Wire Line
+	1100 1300 900  1300
+Wire Wire Line
+	1100 1200 1100 1300
+$Comp
+L +12V #PWR053
+U 1 1 5859BF08
+P 1100 1200
+F 0 "#PWR053" H 1100 1050 50  0001 C CNN
+F 1 "+12V" H 1100 1340 50  0000 C CNN
+F 2 "" H 1100 1200 50  0000 C CNN
+F 3 "" H 1100 1200 50  0000 C CNN
+	1    1100 1200
+	1    0    0    -1
+$EndComp
+$Comp
+L PWR_FLAG #FLG054
+U 1 1 585B5E60
+P 950 1250
+F 0 "#FLG054" H 950 1345 50  0001 C CNN
+F 1 "PWR_FLAG" H 950 1430 50  0000 C CNN
+F 2 "" H 950 1250 50  0000 C CNN
+F 3 "" H 950 1250 50  0000 C CNN
+	1    950  1250
+	1    0    0    -1
+$EndComp
+Wire Wire Line
+	950  1250 950  1300
+Connection ~ 950  1300
+$Comp
+L C C30
+U 1 1 585B97AE
+P 8500 2800
+F 0 "C30" H 8525 2900 50  0000 L CNN
+F 1 "1uF" H 8525 2700 50  0000 L CNN
+F 2 "Capacitors_SMD:C_0603" H 8538 2650 50  0001 C CNN
+F 3 "" H 8500 2800 50  0000 C CNN
+	1    8500 2800
+	1    0    0    -1
+$EndComp
+$Comp
+L GND #PWR055
+U 1 1 585B9832
+P 8500 3050
+F 0 "#PWR055" H 8500 2800 50  0001 C CNN
+F 1 "GND" H 8500 2900 50  0000 C CNN
+F 2 "" H 8500 3050 50  0000 C CNN
+F 3 "" H 8500 3050 50  0000 C CNN
+	1    8500 3050
+	1    0    0    -1
+$EndComp
+Wire Wire Line
+	8500 2950 8500 3050
+Connection ~ 8500 2600
+NoConn ~ 8350 3200
+NoConn ~ 8350 3100
+NoConn ~ 8350 3000
+NoConn ~ 8350 2900
+NoConn ~ 8350 2800
+NoConn ~ 8350 2700
 $EndSCHEMATC

Commit message: Finished PCB
Parts:
- P1: footprint Connectors_JST:JST_PH_B2B-PH-K_02x2.00mm_Straight -> Connect:PINHEAD1-2
Changed lines of the file:
@@
 F 0 "P1" H 5150 3300 50  0000 C CNN
 F 1 "CONN_01X02" V 5250 3150 50  0000 C CNN
-F 2 "Connectors_JST:JST_PH_B2B-PH-K_02x2.00mm_Straight" H 5150 3150 50  0001 C CNN
+F 2 "Connect:PINHEAD1-2" H 5150 3150 50  0001 C CNN
 F 3 "" H 5150 3150 50  0000 C CNN
 	1    5150 3150
