File: Electrical/LED_Snowboard.sch (KiCad schematic (older format))
At the start: 0 parts

Commit message: Continued work on schematic
Changed lines of the file:
@@
 F3 "I2C_SDA" I L 8100 2950 60
 F4 "I2C_SCL" I L 8100 3050 60
+F5 "UART_RX_Sen" I L 8100 3150 60
+F6 "UART_TX_Sen" I L 8100 3250 60
 $EndSheet
 $Sheet

Commit message: schematic 95% donbe
Changed lines of the file:
@@
 F6 "UART_RX" I L 5050 3250 60
 F7 "UART_TX" I L 5050 3350 60
-F8 "BAT_MON" I L 5050 3450 60
+F8 "BAT_MON" I R 7300 4700 60
+F9 "BAT_Volt" I L 5050 3450 60
 $EndSheet
 $Sheet
-S 1700 2800 2250 2000
+S 1000 2800 2250 2000
 U 584334CD
 F0 "Power Supply" 60
 F1 "PWR.sch" 60
-F2 "BAT_IN" I R 3950 3050 60
-F3 "V_IN" I R 3950 2900 60
-F4 "5V_OUT" I R 3950 3300 60
-F5 "3.3V_OUT" I R 3950 3200 60
+F2 "BAT_IN" I R 3250 3050 60
+F3 "V_IN" I R 3250 2900 60
+F4 "5V_OUT" I R 3250 3300 60
+F5 "3.3V_OUT" I R 3250 3200 60
+F6 "V_SYS" I L 1000 3450 60
+F7 "VREF" I L 1000 3550 60
+F8 "TS" I L 1000 3650 60
+F9 "AVCC" I L 1000 3750 60
+F10 "OVPSET" I L 1000 3850 60
+F11 "BAT_Volt" I R 3250 3450 60
 $EndSheet
 $Sheet
-S 8100 2750 2250 2000
+S 8650 2750 2250 2000
 U 584339A7
 F0 "Sensors" 60
 F1 "Sensors.sch" 60
-F2 "3.3V_IN" I L 8100 2850 60
-F3 "I2C_SDA" I L 8100 2950 60
-F4 "I2C_SCL" I L 8100 3050 60
-F5 "UART_RX_Sen" I L 8100 3150 60
-F6 "UART_TX_Sen" I L 8100 3250 60
+F2 "3.3V_IN" I L 8650 2850 60
+F3 "I2C_SDA" I L 8650 2950 60
+F4 "I2C_SCL" I L 8650 3050 60
+F5 "UART_RX_Sen" I L 8650 3150 60
+F6 "UART_TX_Sen" I L 8650 3250 60
 $EndSheet
 $Sheet
-S 1700 5150 2250 2000
+S 1000 5150 2250 2000
 U 584339AE
 F0 "Connectors" 60
 F1 "Connectors.sch" 60
-F2 "BAT_IN" I R 3950 5250 60
-F3 "V_IN" I R 3950 5350 60
-F4 "5V_IN" I R 3950 5450 60
-F5 "LED_CTRL" I R 3950 5550 60
-F6 "3.3V_IN" I R 3950 5650 60
-F7 "I2C_SDA" I R 3950 5750 60
-F8 "I2C_SCL" I R 3950 5850 60
-F9 "DISP_RST" I R 3950 5950 60
+F2 "BAT_IN" I R 3250 5250 60
+F3 "V_IN" I R 3250 5350 60
+F4 "5V_IN" I R 3250 5450 60
+F5 "LED_CTRL" I R 3250 5550 60
+F6 "3.3V_IN" I R 3250 5650 60
+F7 "I2C_SDA" I R 3250 5750 60
+F8 "I2C_SCL" I R 3250 5850 60
+F9 "DISP_RST" I R 3250 5950 60
 $EndSheet
+Text HLabel 3400 5550 2    60   Input ~ 0
+LED_CTRL_Conn
+Text HLabel 4900 3150 0    60   Input ~ 0
+LED_CTRL_Conn
+Text HLabel 3400 5650 2    60   Input ~ 0
+3.3V
+Text HLabel 8500 2850 0    60   Input ~ 0
+3.3V
+Text HLabel 4900 3350 0    60   Input ~ 0
+UART_TX_RX
+Text HLabel 4900 3250 0    60   Input ~ 0
+UART_RX_TX
+Text HLabel 4900 2850 0    60   Input ~ 0
+I2C_SDA_Conn
+Text HLabel 4900 2950 0    60   Input ~ 0
+I2C_SCL_Conn
+Text HLabel 8500 2950 0    60   Input ~ 0
+I2C_SDA_Conn
+Text HLabel 8500 3050 0    60   Input ~ 0
+I2C_SCL_Conn
+Wire Wire Line
+	8500 3050 8650 3050
+Wire Wire Line
+	8650 2950 8500 2950
+Wire Wire Line
+	8500 2850 8650 2850
+Text HLabel 3350 3200 2    60   Input ~ 0
+3.3V
+Wire Wire Line
+	3350 3200 3250 3200
+Text HLabel 3350 3300 2    60   Input ~ 0
+5V
+Wire Wire Line
+	3350 3300 3250 3300
+Wire Wire Line
+	3400 5650 3250 5650
+Text HLabel 3400 5450 2    60   Input ~ 0
+5V
+Wire Wire Line
+	3400 5450 3250 5450
+Wire Wire Line
+	3400 5550 3250 5550
+Text HLabel 3400 5250 2    60   Input ~ 0
+BAT
+Text HLabel 3350 2900 2    60   Input ~ 0
+V_IN_Conn
+Wire Wire Line
+	3350 2900 3250 2900
+Text HLabel 3400 5350 2    60   Input ~ 0
+V_IN_Conn
+Wire Wire Line
+	3400 5350 3250 5350
+Wire Wire Line
+	3400 5250 3250 5250
+Text HLabel 3350 3050 2    60   Input ~ 0
+BAT
+Wire Wire Line
+	3350 3050 3250 3050
+Text HLabel 3400 5750 2    60   Input ~ 0
+I2C_SDA_Conn
+Text HLabel 3400 5850 2    60   Input ~ 0
+I2C_SCL_Conn
+Text HLabel 4900 3050 0    60   Input ~ 0
+DISP_RST_Conn
+Text HLabel 3400 5950 2    60   Input ~ 0
+DISP_RST_Conn
+Text HLabel 8500 3250 0    60   Input ~ 0
+UART_RX_TX
+Text HLabel 8500 3150 0    60   Input ~ 0
+UART_TX_RX
+Wire Wire Line
+	8650 3150 8500 3150
+Wire Wire Line
+	8500 3250 8650 3250
+Wire Wire Line
+	4900 3350 5050 3350
+Wire Wire Line
+	5050 3250 4900 3250
+Wire Wire Line
+	4900 3150 5050 3150
+Wire Wire Line
+	5050 3050 4900 3050
+Wire Wire Line
+	4900 2950 5050 2950
+Wire Wire Line
+	5050 2850 4900 2850
+Wire Wire Line
+	3400 5950 3250 5950
+Wire Wire Line
+	3250 5850 3400 5850
+Wire Wire Line
+	3250 5750 3400 5750
+Text HLabel 3350 3450 2    60   Input ~ 0
+BAT_V
+Text HLabel 4900 3450 0    60   Input ~ 0
+BAT_V
+Wire Wire Line
+	5050 3450 4900 3450
+Wire Wire Line
+	3350 3450 3250 3450
 $EndSCHEMATC
