File: Electrical/MCU.sch (KiCad schematic (older format))
At the start: 3 parts

Commit message: almost finished with MCU sheet
Parts:
- gave numbers to parts that had none: 3
Connections:
- net DISP_RST: now also U1.39 (17)
- net LED_CTRL: now also U1.38 (16)
- net UART_RX: now also U1.2 (0)
- net UART_TX: now also U1.3 (1)
Changed lines of the file:
@@
 $EndDescr
 $Comp
-L Teensy_3.6 U?
+L Teensy_3.6 U1
 U 1 1 58430E2B
 P 7700 3000
-F 0 "U?" H 7700 2800 50  0000 C CNN
+F 0 "U1" H 7700 2800 50  0000 C CNN
 F 1 "Teensy_3.6" H 7700 3000 50  0000 C CNN
 F 2 "MODULE" H 8000 1500 50  0001 C CNN
@@
 1A 89 BE 04 41 10 04 51 D7 48 F4 25 08 82 20 88 BA 46 A2 2F 41 10 04 41 D4 35 12 7D 09 82 20 08
 A2 AE 91 E8 4B 10 04 41 10 75 ED FF 01 D0 70 D0 C9 E7 A1 7F 24 00 00 00 00 49 45 4E 44 AE 42 60
-82 58
+82 02
 EndData
 $EndBitmap
 $Comp
-L +3.3V #PWR?
+L +3.3V #PWR2
 U 1 1 58430F11
 P 8900 1850
-F 0 "#PWR?" H 8900 1700 50  0001 C CNN
+F 0 "#PWR2" H 8900 1700 50  0001 C CNN
 F 1 "+3.3V" H 8900 1990 50  0000 C CNN
 F 2 "" H 8900 1850 50  0000 C CNN
@@
 $EndComp
 $Comp
-L GND #PWR?
+L GND #PWR1
 U 1 1 58430F27
-P 6600 2050
-F 0 "#PWR?" H 6600 1800 50  0001 C CNN
-F 1 "GND" H 6600 1900 50  0000 C CNN
-F 2 "" H 6600 2050 50  0000 C CNN
-F 3 "" H 6600 2050 50  0000 C CNN
-	1    6600 2050
+P 6050 2050
+F 0 "#PWR1" H 6050 1800 50  0001 C CNN
+F 1 "GND" H 6050 1900 50  0000 C CNN
+F 2 "" H 6050 2050 50  0000 C CNN
+F 3 "" H 6050 2050 50  0000 C CNN
+	1    6050 2050
 	1    0    0    -1
 $EndComp
 $Comp
-L GND #PWR?
+L GND #PWR3
 U 1 1 58430F3C
 P 8900 3450
-F 0 "#PWR?" H 8900 3200 50  0001 C CNN
+F 0 "#PWR3" H 8900 3200 50  0001 C CNN
 F 1 "GND" H 8900 3300 50  0000 C CNN
 F 2 "" H 8900 3450 50  0000 C CNN
@@
 	8900 3350 8450 3350
 Wire Wire Line
-	6950 1950 6600 1950
+	6050 1950 6950 1950
 Wire Wire Line
-	6600 1950 6600 2050
+	6050 1950 6050 2050
 Wire Wire Line
 	8450 1950 8900 1950
@@
 	8450 2750 9100 2750
 $Comp
-L R R?
+L R R2
 U 1 1 5843107B
 P 9000 2450
-F 0 "R?" V 9080 2450 50  0000 C CNN
+F 0 "R2" V 9080 2450 50  0000 C CNN
 F 1 "4.7k" V 9000 2450 50  0000 C CNN
 F 2 "" V 8930 2450 50  0000 C CNN
@@
 $EndComp
 $Comp
-L R R?
+L R R1
 U 1 1 584310B0
 P 8850 2450
-F 0 "R?" V 8930 2450 50  0000 C CNN
+F 0 "R1" V 8930 2450 50  0000 C CNN
 F 1 "4.7k" V 8850 2450 50  0000 C CNN
 F 2 "" V 8780 2450 50  0000 C CNN
@@
 Text HLabel 9100 2950 2    60   Input ~ 0
 LED_CTRL
-Text HLabel 9100 3050 2    60   Input ~ 0
+Text HLabel 6700 2050 0    60   Input ~ 0
 UART_RX
-Text HLabel 9100 3150 2    60   Input ~ 0
+Text HLabel 6700 2150 0    60   Input ~ 0
 UART_TX
-Text HLabel 9100 3250 2    60   Input ~ 0
+Text HLabel 9100 3050 2    60   Input ~ 0
 BAT_MON
+Wire Wire Line
+	6950 2050 6700 2050
+Wire Wire Line
+	6700 2150 6950 2150
+Wire Wire Line
+	9100 2850 8450 2850
+Wire Wire Line
+	9100 2950 8450 2950
 $EndSCHEMATC

Commit message: schematic 95% donbe
Parts:
- added C29: C, Capacitors_SMD:C_0603, symbol C
- added R25, R26: R, Capacitors_SMD:C_0603, symbol R
- R1, R2: footprint (none) -> Resistors_SMD:R_0603
Connections:
- net BAT_MON: now also U1.37 (15), C29.1, R25.2, R26.1
- net GND: now also C29.2, R26.2
- new net BAT_Volt: R25.1
Other:
- note added: "This seems very simple...."
Changed lines of the file:
@@
 1A 89 BE 04 41 10 04 51 D7 48 F4 25 08 82 20 88 BA 46 A2 2F 41 10 04 41 D4 35 12 7D 09 82 20 08
 A2 AE 91 E8 4B 10 04 41 10 75 ED FF 01 D0 70 D0 C9 E7 A1 7F 24 00 00 00 00 49 45 4E 44 AE 42 60
-82 02
+82 00
 EndData
 $EndBitmap
 $Comp
-L +3.3V #PWR2
+L +3.3V #PWR01
 U 1 1 58430F11
 P 8900 1850
-F 0 "#PWR2" H 8900 1700 50  0001 C CNN
+F 0 "#PWR01" H 8900 1700 50  0001 C CNN
 F 1 "+3.3V" H 8900 1990 50  0000 C CNN
 F 2 "" H 8900 1850 50  0000 C CNN
@@
 $EndComp
 $Comp
-L GND #PWR1
+L GND #PWR02
 U 1 1 58430F27
 P 6050 2050
-F 0 "#PWR1" H 6050 1800 50  0001 C CNN
+F 0 "#PWR02" H 6050 1800 50  0001 C CNN
 F 1 "GND" H 6050 1900 50  0000 C CNN
 F 2 "" H 6050 2050 50  0000 C CNN
@@
 $EndComp
 $Comp
-L GND #PWR3
+L GND #PWR03
 U 1 1 58430F3C
 P 8900 3450
-F 0 "#PWR3" H 8900 3200 50  0001 C CNN
+F 0 "#PWR03" H 8900 3200 50  0001 C CNN
 F 1 "GND" H 8900 3300 50  0000 C CNN
 F 2 "" H 8900 3450 50  0000 C CNN
@@
 F 0 "R2" V 9080 2450 50  0000 C CNN
 F 1 "4.7k" V 9000 2450 50  0000 C CNN
-F 2 "" V 8930 2450 50  0000 C CNN
+F 2 "Resistors_SMD:R_0603" V 8930 2450 50  0001 C CNN
 F 3 "" H 9000 2450 50  0000 C CNN
 	1    9000 2450
@@
 F 0 "R1" V 8930 2450 50  0000 C CNN
 F 1 "4.7k" V 8850 2450 50  0000 C CNN
-F 2 "" V 8780 2450 50  0000 C CNN
+F 2 "Resistors_SMD:R_0603" V 8780 2450 50  0001 C CNN
 F 3 "" H 8850 2450 50  0000 C CNN
 	1    8850 2450
@@
 Wire Wire Line
 	9100 2950 8450 2950
+Text HLabel 4650 2850 0    60   Input ~ 0
+BAT_Volt
+Wire Wire Line
+	9100 3050 8450 3050
+Text HLabel 5550 3400 2    60   Input ~ 0
+BAT_MON
+$Comp
+L R R25
+U 1 1 585BA5FA
+P 4850 3150
+F 0 "R25" V 4930 3150 50  0000 C CNN
+F 1 "R" V 4850 3150 50  0000 C CNN
+F 2 "Capacitors_SMD:C_0603" V 4780 3150 50  0001 C CNN
+F 3 "" H 4850 3150 50  0000 C CNN
+	1    4850 3150
+	1    0    0    -1
+$EndComp
+$Comp
+L R R26
+U 1 1 585BA64B
+P 4850 3650
+F 0 "R26" V 4930 3650 50  0000 C CNN
+F 1 "R" V 4850 3650 50  0000 C CNN
+F 2 "Capacitors_SMD:C_0603" V 4780 3650 50  0001 C CNN
+F 3 "" H 4850 3650 50  0000 C CNN
+	1    4850 3650
+	1    0    0    -1
+$EndComp
+$Comp
+L C C29
+U 1 1 585BA67B
+P 5250 3650
+F 0 "C29" H 5275 3750 50  0000 L CNN
+F 1 "C" H 5275 3550 50  0000 L CNN
+F 2 "Capacitors_SMD:C_0603" H 5288 3500 50  0001 C CNN
+F 3 "" H 5250 3650 50  0000 C CNN
+	1    5250 3650
+	1    0    0    -1
+$EndComp
+Wire Wire Line
+	4850 3300 4850 3500
+Wire Wire Line
+	4850 3400 5550 3400
+Connection ~ 4850 3400
+Wire Wire Line
+	5250 3500 5250 3400
+Connection ~ 5250 3400
+Wire Wire Line
+	4850 3800 4850 4000
+Wire Wire Line
+	4850 3900 5250 3900
+Wire Wire Line
+	5250 3900 5250 3800
+Connection ~ 4850 3900
+$Comp
+L GND #PWR04
+U 1 1 585BA9C4
+P 4850 4000
+F 0 "#PWR04" H 4850 3750 50  0001 C CNN
+F 1 "GND" H 4850 3850 50  0000 C CNN
+F 2 "" H 4850 4000 50  0000 C CNN
+F 3 "" H 4850 4000 50  0000 C CNN
+	1    4850 4000
+	1    0    0    -1
+$EndComp
+Wire Wire Line
+	4650 2850 4850 2850
+Wire Wire Line
+	4850 2850 4850 3000
+Text Notes 4400 2700 0    60   ~ 0
+This seems very simple....
 $EndSCHEMATC

Commit message: minor tweaks
Parts:
- R25, R26: footprint Capacitors_SMD:C_0603 -> Resistors_SMD:R_0603
- U1: footprint MODULE -> Snow_parts:Teensy-3.6
Changed lines of the file:
@@
 F 0 "U1" H 7700 2800 50  0000 C CNN
 F 1 "Teensy_3.6" H 7700 3000 50  0000 C CNN
-F 2 "MODULE" H 8000 1500 50  0001 C CNN
+F 2 "Snow_parts:Teensy-3.6" H 8000 1500 50  0001 C CNN
 F 3 "DOCUMENTATION" H 7850 1600 50  0001 C CNN
 	1    7700 3000
@@
 1A 89 BE 04 41 10 04 51 D7 48 F4 25 08 82 20 88 BA 46 A2 2F 41 10 04 41 D4 35 12 7D 09 82 20 08
 A2 AE 91 E8 4B 10 04 41 10 75 ED FF 01 D0 70 D0 C9 E7 A1 7F 24 00 00 00 00 49 45 4E 44 AE 42 60
-82 78
+82 00
 EndData
 $EndBitmap
@@
 F 0 "R25" V 4930 3150 50  0000 C CNN
 F 1 "R" V 4850 3150 50  0000 C CNN
-F 2 "Capacitors_SMD:C_0603" V 4780 3150 50  0001 C CNN
+F 2 "Resistors_SMD:R_0603" V 4780 3150 50  0001 C CNN
 F 3 "" H 4850 3150 50  0000 C CNN
 	1    4850 3150
@@
 F 0 "R26" V 4930 3650 50  0000 C CNN
 F 1 "R" V 4850 3650 50  0000 C CNN
-F 2 "Capacitors_SMD:C_0603" V 4780 3650 50  0001 C CNN
+F 2 "Resistors_SMD:R_0603" V 4780 3650 50  0001 C CNN
 F 3 "" H 4850 3650 50  0000 C CNN
 	1    4850 3650

Commit message: Minor Changes
Parts:
- C29: value C -> 1uF
- R25: value R -> 10K
- R26: value R -> 36K
Changed lines of the file:
@@
 P 4850 3150
 F 0 "R25" V 4930 3150 50  0000 C CNN
-F 1 "R" V 4850 3150 50  0000 C CNN
+F 1 "10K" V 4850 3150 50  0000 C CNN
 F 2 "Resistors_SMD:R_0603" V 4780 3150 50  0001 C CNN
 F 3 "" H 4850 3150 50  0000 C CNN
@@
 P 4850 3650
 F 0 "R26" V 4930 3650 50  0000 C CNN
-F 1 "R" V 4850 3650 50  0000 C CNN
+F 1 "36K" V 4850 3650 50  0000 C CNN
 F 2 "Resistors_SMD:R_0603" V 4780 3650 50  0001 C CNN
 F 3 "" H 4850 3650 50  0000 C CNN
@@
 P 5250 3650
 F 0 "C29" H 5275 3750 50  0000 L CNN
-F 1 "C" H 5275 3550 50  0000 L CNN
+F 1 "1uF" H 5275 3550 50  0000 L CNN
 F 2 "Capacitors_SMD:C_0603" H 5288 3500 50  0001 C CNN
 F 3 "" H 5250 3650 50  0000 C CNN
