File: Electrical/PWR.sch (KiCad schematic (older format))
At the start: 55 parts, among them Q1 CSD17313Q2, U2 TPS63021, U3 TPS61236, U4 BQ24170

Commit message: Finished PCB
Changed lines of the file:
@@
 	7050 2400 7050 2700
 Wire Wire Line
-	8950 2700 7050 2700
+	7050 2700 8950 2700
 Connection ~ 8950 2050
 Wire Wire Line
@@
 	4450 6050 4700 6050
 Wire Wire Line
-	4700 5750 4700 6050
+	4700 6050 4700 5750
 Wire Wire Line
 	4450 5750 6250 5750
@@
 $EndComp
 Wire Wire Line
-	8950 1800 8950 2700
+	8950 2700 8950 1800
 Connection ~ 10300 1300
 Wire Wire Line

Commit message: really minor commit to keep everything together
Parts:
- D1, D2, D3: symbol LED -> LED-RESCUE-LED_Snowboard
Changed lines of the file:
@@
 EESchema Schematic File Version 2
+LIBS:LED_Snowboard-rescue
 LIBS:power
 LIBS:device
@@
 LIBS:contrib
 LIBS:valves
-LIBS:parts
 LIBS:Snowboard_Parts
 LIBS:LED_Snowboard-cache
@@
 V_SYS
 $Comp
-L LED D1
+L LED-RESCUE-LED_Snowboard D1
 U 1 1 58479A9B
 P 4800 2600
@@
 $EndComp
 $Comp
-L LED D3
+L LED-RESCUE-LED_Snowboard D3
 U 1 1 584992A0
 P 6250 4750
@@
 Connection ~ 6250 4200
 $Comp
-L LED D2
+L LED-RESCUE-LED_Snowboard D2
 U 1 1 58499F2B
 P 5700 6400
