File: Electrical/Sensors.sch (KiCad schematic (older format))
At the start: 2 parts

Commit message: Finished sensor sheet
Parts:
- added C? (x2): 0.1uF, symbol C
- added C? (x2): 10uF, symbol C
- added U?: VenusGPS, MODULE, symbol VenusGPS
- C21: renamed from C?; value C -> 10nF
- gave numbers to parts that had none: 1
Connections:
- net +3V3: now also U5.1 (VDDIO), U5.22 (VDD), U5.23 (VDD), U5.3 (VDDIO), U5.7 (CS_A/G), U5.8 (CS_M), C?.1, C?.1, C?.1, U?.7 (3.3V)
- net GND: now also C21.2, U5.14 (RES), U5.15 (RES), U5.16 (RES), U5.17 (RES), U5.18 (RES), U5.19 (GND), U5.20 (GND), U5.5 (SDO_A/G), U5.6 (SDO_M), C?.2, C?.2, C?.2, C?.2, U?.10 (GND), U?.8 (GND)
- net I2C_SCL: now also U5.2 (SCL/SPC)
- net I2C_SDA: now also U5.4 (SDA/SDI/SDO)
- net at U5.21 (CAP): now also C21.1
- net at U5.24 (C1): now also C?.1
- new net UART_RX_Sen: U?.6 (TX0)
- new net UART_TX_Sen: U?.5 (RX0)
Other:
- note added: "9DoF IMU"
- note added: "GPS Module"
- moved on the sheet: C21, U5

Commit message: schematic 95% donbe
Parts:
- C21: footprint (none) -> Capacitors_SMD:C_0603
- C25, C26, C27, C28: renamed from C?; footprint (none) -> Capacitors_SMD:C_0603
- U5: footprint MODULE -> SPEX_Parts:LGA-24
- gave numbers to parts that had none: 1
Connections:
- net UART_RX_Sen: now also U6.5 (RX0); no longer U6.6 (TX0)
- net UART_TX_Sen: now also U6.6 (TX0); no longer U6.5 (RX0)
Changed lines of the file:
@@
 F 0 "U5" H 7400 4150 50  0000 C CNN
 F 1 "LSM9DS1" H 7400 4250 50  0000 C CNN
-F 2 "MODULE" H 7550 2850 50  0001 C CNN
+F 2 "SPEX_Parts:LGA-24" H 7550 2850 50  0001 C CNN
 F 3 "DOCUMENTATION" H 7550 2850 50  0001 C CNN
 	1    7400 3550
@@
 F 0 "C21" H 8825 3650 50  0000 L CNN
 F 1 "10nF" H 8825 3450 50  0000 L CNN
-F 2 "" H 8838 3400 50  0000 C CNN
+F 2 "Capacitors_SMD:C_0603" H 8838 3400 50  0001 C CNN
 F 3 "" H 8800 3550 50  0000 C CNN
 	1    8800 3550
@@
 $EndComp
 $Comp
-L +3.3V #PWR21
+L +3.3V #PWR025
 U 1 1 584A16CD
 P 1300 900
-F 0 "#PWR21" H 1300 750 50  0001 C CNN
+F 0 "#PWR025" H 1300 750 50  0001 C CNN
 F 1 "+3.3V" H 1300 1040 50  0000 C CNN
 F 2 "" H 1300 900 50  0000 C CNN
@@
 3.3V_IN
 $Comp
-L +3.3V #PWR23
+L +3.3V #PWR026
 U 1 1 584A1716
 P 5950 2750
-F 0 "#PWR23" H 5950 2600 50  0001 C CNN
+F 0 "#PWR026" H 5950 2600 50  0001 C CNN
 F 1 "+3.3V" H 5950 2890 50  0000 C CNN
 F 2 "" H 5950 2750 50  0000 C CNN
@@
 $EndComp
 $Comp
-L GND #PWR22
+L GND #PWR027
 U 1 1 584A17B5
 P 5950 4400
-F 0 "#PWR22" H 5950 4150 50  0001 C CNN
+F 0 "#PWR027" H 5950 4150 50  0001 C CNN
 F 1 "GND" H 5950 4250 50  0000 C CNN
 F 2 "" H 5950 4400 50  0000 C CNN
@@
 I2C_SCL
 $Comp
-L C C?
+L C C28
 U 1 1 5859EA8D
 P 9150 3550
-F 0 "C?" H 9175 3650 50  0000 L CNN
+F 0 "C28" H 9175 3650 50  0000 L CNN
 F 1 "0.1uF" H 9175 3450 50  0000 L CNN
-F 2 "" H 9188 3400 50  0000 C CNN
+F 2 "Capacitors_SMD:C_0603" H 9188 3400 50  0001 C CNN
 F 3 "" H 9150 3550 50  0000 C CNN
 	1    9150 3550
@@
 $EndComp
 $Comp
-L GND #PWR?
+L GND #PWR028
 U 1 1 5859EBFA
 P 8350 4400
-F 0 "#PWR?" H 8350 4150 50  0001 C CNN
+F 0 "#PWR028" H 8350 4150 50  0001 C CNN
 F 1 "GND" H 8350 4250 50  0000 C CNN
 F 2 "" H 8350 4400 50  0000 C CNN
@@
 $EndComp
 $Comp
-L +3.3V #PWR?
+L +3.3V #PWR029
 U 1 1 5859ECA7
 P 8500 2750
-F 0 "#PWR?" H 8500 2600 50  0001 C CNN
+F 0 "#PWR029" H 8500 2600 50  0001 C CNN
 F 1 "+3.3V" H 8500 2890 50  0000 C CNN
 F 2 "" H 8500 2750 50  0000 C CNN
@@
 $EndComp
 $Comp
-L C C?
+L C C27
 U 1 1 5859EECC
 P 8500 3550
-F 0 "C?" H 8525 3650 50  0000 L CNN
+F 0 "C27" H 8525 3650 50  0000 L CNN
 F 1 "10uF" H 8525 3450 50  0000 L CNN
-F 2 "" H 8538 3400 50  0000 C CNN
+F 2 "Capacitors_SMD:C_0603" H 8538 3400 50  0001 C CNN
 F 3 "" H 8500 3550 50  0000 C CNN
 	1    8500 3550
@@
 $EndComp
 $Comp
-L C C?
+L C C26
 U 1 1 5859EF97
 P 5950 3550
-F 0 "C?" H 5975 3650 50  0000 L CNN
+F 0 "C26" H 5975 3650 50  0000 L CNN
 F 1 "0.1uF" H 5975 3450 50  0000 L CNN
-F 2 "" H 5988 3400 50  0000 C CNN
+F 2 "Capacitors_SMD:C_0603" H 5988 3400 50  0001 C CNN
 F 3 "" H 5950 3550 50  0000 C CNN
 	1    5950 3550
@@
 	8150 3500 8350 3500
 Wire Wire Line
-	8350 3400 8350 3500
-Wire Wire Line
-	8350 3500 8350 3600
-Wire Wire Line
-	8350 3600 8350 3700
-Wire Wire Line
-	8350 3700 8350 3800
-Wire Wire Line
-	8350 3800 8350 3900
-Wire Wire Line
-	8350 3900 8350 4000
-Wire Wire Line
-	8350 4000 8350 4300
-Wire Wire Line
-	8350 4300 8350 4400
+	8350 3400 8350 4400
 Wire Wire Line
 	8150 4000 8350 4000
@@
 	8800 4300 8800 3700
 Wire Wire Line
-	8350 4300 8500 4300
-Wire Wire Line
-	8500 4300 8800 4300
-Wire Wire Line
-	8800 4300 9150 4300
+	8350 4300 9150 4300
 Connection ~ 8350 4300
 Wire Wire Line
@@
 Connection ~ 8800 4300
 Wire Wire Line
-	8500 2750 8500 3100
-Wire Wire Line
-	8500 3100 8500 3200
-Wire Wire Line
-	8500 3200 8500 3400
+	8500 2750 8500 3400
 Wire Wire Line
 	8500 3100 8150 3100
@@
 Connection ~ 8500 4300
 Wire Wire Line
-	5950 2750 5950 3000
-Wire Wire Line
-	5950 3000 5950 3200
-Wire Wire Line
-	5950 3200 5950 3400
-Wire Wire Line
-	5950 3000 6550 3000
-Wire Wire Line
-	6550 3000 6650 3000
-Wire Wire Line
-	5700 3200 5950 3200
-Wire Wire Line
-	5950 3200 6650 3200
+	5950 2750 5950 3400
+Wire Wire Line
+	5950 3000 6650 3000
+Wire Wire Line
+	5700 3200 6650 3200
 Connection ~ 5950 3000
 Wire Wire Line
-	5950 3700 5950 4350
-Wire Wire Line
-	5950 4350 5950 4400
+	5950 3700 5950 4400
 Connection ~ 5950 3200
 $Comp
-L C C?
+L C C25
 U 1 1 5859F28B
 P 5700 3550
-F 0 "C?" H 5725 3650 50  0000 L CNN
+F 0 "C25" H 5725 3650 50  0000 L CNN
 F 1 "10uF" H 5725 3450 50  0000 L CNN
-F 2 "" H 5738 3400 50  0000 C CNN
+F 2 "Capacitors_SMD:C_0603" H 5738 3400 50  0001 C CNN
 F 3 "" H 5700 3550 50  0000 C CNN
 	1    5700 3550
@@
 	5700 3700 5700 4350
 Wire Wire Line
-	5700 4350 5950 4350
-Wire Wire Line
-	5950 4350 6600 4350
+	5700 4350 6600 4350
 Connection ~ 5950 4350
 Wire Wire Line
@@
 	6550 3700 6650 3700
 Wire Wire Line
-	6550 3000 6550 3600
-Wire Wire Line
-	6550 3600 6550 3700
+	6550 3000 6550 3700
 Connection ~ 6550 3000
 Wire Wire Line
@@
 	6650 3500 6600 3500
 Wire Wire Line
-	6600 4350 6600 3500
-Wire Wire Line
-	6600 3500 6600 3400
+	6600 4350 6600 3400
 Wire Wire Line
 	6600 3400 6650 3400
 Connection ~ 6600 3500
 $Comp
-L VenusGPS U?
+L VenusGPS U6
 U 1 1 5859FDE2
 P 4050 3400
-F 0 "U?" H 4050 3150 50  0000 C CNN
+F 0 "U6" H 4050 3150 50  0000 C CNN
 F 1 "VenusGPS" H 4050 3600 50  0000 C CNN
 F 2 "MODULE" H 4350 2700 50  0001 C CNN
@@
 	1    0    0    -1
 $EndComp
+Text HLabel 3250 3600 0    60   Input ~ 0
+UART_RX_Sen
 Text HLabel 3250 3700 0    60   Input ~ 0
-UART_RX_Sen
-Text HLabel 3250 3600 0    60   Input ~ 0
 UART_TX_Sen
 Wire Wire Line
@@
 	3300 3700 3250 3700
 $Comp
-L +3.3V #PWR?
+L +3.3V #PWR030
 U 1 1 585A087F
 P 2450 3750
-F 0 "#PWR?" H 2450 3600 50  0001 C CNN
+F 0 "#PWR030" H 2450 3600 50  0001 C CNN
 F 1 "+3.3V" H 2450 3890 50  0000 C CNN
 F 2 "" H 2450 3750 50  0000 C CNN
@@
 	2450 3800 2450 3750
 $Comp
-L GND #PWR?
+L GND #PWR031
 U 1 1 585A0A36
 P 2450 3950
-F 0 "#PWR?" H 2450 3700 50  0001 C CNN
+F 0 "#PWR031" H 2450 3700 50  0001 C CNN
 F 1 "GND" H 2450 3800 50  0000 C CNN
 F 2 "" H 2450 3950 50  0000 C CNN
@@
 	2450 3900 3300 3900
 $Comp
-L GND #PWR?
+L GND #PWR032
 U 1 1 585A0BD3
 P 4950 3950
-F 0 "#PWR?" H 4950 3700 50  0001 C CNN
+F 0 "#PWR032" H 4950 3700 50  0001 C CNN
 F 1 "GND" H 4950 3800 50  0000 C CNN
 F 2 "" H 4950 3950 50  0000 C CNN

Commit message: minor tweaks
Parts:
- U6: footprint MODULE -> Snow_parts:VenusGPS
Changed lines of the file:
@@
 $EndComp
 $Comp
-L +3.3V #PWR025
+L +3.3V #PWR026
 U 1 1 584A16CD
 P 1300 900
-F 0 "#PWR025" H 1300 750 50  0001 C CNN
+F 0 "#PWR026" H 1300 750 50  0001 C CNN
 F 1 "+3.3V" H 1300 1040 50  0000 C CNN
 F 2 "" H 1300 900 50  0000 C CNN
@@
 3.3V_IN
 $Comp
-L +3.3V #PWR026
+L +3.3V #PWR027
 U 1 1 584A1716
 P 5950 2750
-F 0 "#PWR026" H 5950 2600 50  0001 C CNN
+F 0 "#PWR027" H 5950 2600 50  0001 C CNN
 F 1 "+3.3V" H 5950 2890 50  0000 C CNN
 F 2 "" H 5950 2750 50  0000 C CNN
@@
 $EndComp
 $Comp
-L GND #PWR027
+L GND #PWR028
 U 1 1 584A17B5
 P 5950 4400
-F 0 "#PWR027" H 5950 4150 50  0001 C CNN
+F 0 "#PWR028" H 5950 4150 50  0001 C CNN
 F 1 "GND" H 5950 4250 50  0000 C CNN
 F 2 "" H 5950 4400 50  0000 C CNN
@@
 $EndComp
 $Comp
-L GND #PWR028
+L GND #PWR029
 U 1 1 5859EBFA
 P 8350 4400
-F 0 "#PWR028" H 8350 4150 50  0001 C CNN
+F 0 "#PWR029" H 8350 4150 50  0001 C CNN
 F 1 "GND" H 8350 4250 50  0000 C CNN
 F 2 "" H 8350 4400 50  0000 C CNN
@@
 $EndComp
 $Comp
-L +3.3V #PWR029
+L +3.3V #PWR030
 U 1 1 5859ECA7
 P 8500 2750
-F 0 "#PWR029" H 8500 2600 50  0001 C CNN
+F 0 "#PWR030" H 8500 2600 50  0001 C CNN
 F 1 "+3.3V" H 8500 2890 50  0000 C CNN
 F 2 "" H 8500 2750 50  0000 C CNN
@@
 F 0 "U6" H 4050 3150 50  0000 C CNN
 F 1 "VenusGPS" H 4050 3600 50  0000 C CNN
-F 2 "MODULE" H 4350 2700 50  0001 C CNN
+F 2 "Snow_parts:VenusGPS" H 4350 2700 50  0001 C CNN
 F 3 "DOCUMENTATION" H 4200 2800 50  0001 C CNN
 	1    4050 3400
@@
 	3300 3700 3250 3700
 $Comp
-L +3.3V #PWR030
+L +3.3V #PWR031
 U 1 1 585A087F
 P 2450 3750
-F 0 "#PWR030" H 2450 3600 50  0001 C CNN
+F 0 "#PWR031" H 2450 3600 50  0001 C CNN
 F 1 "+3.3V" H 2450 3890 50  0000 C CNN
 F 2 "" H 2450 3750 50  0000 C CNN
@@
 	2450 3800 2450 3750
 $Comp
-L GND #PWR031
+L GND #PWR032
 U 1 1 585A0A36
 P 2450 3950
-F 0 "#PWR031" H 2450 3700 50  0001 C CNN
+F 0 "#PWR032" H 2450 3700 50  0001 C CNN
 F 1 "GND" H 2450 3800 50  0000 C CNN
 F 2 "" H 2450 3950 50  0000 C CNN
@@
 	2450 3900 3300 3900
 $Comp
-L GND #PWR032
+L GND #PWR033
 U 1 1 585A0BD3
 P 4950 3950
-F 0 "#PWR032" H 4950 3700 50  0001 C CNN
+F 0 "#PWR033" H 4950 3700 50  0001 C CNN
 F 1 "GND" H 4950 3800 50  0000 C CNN
 F 2 "" H 4950 3950 50  0000 C CNN
